File: nrom-board/nrom-board-rounded.kicad_pcb (KiCad board)
At the start: 2 copper layers, 90 x 56.8 mm, 12 parts, among them J1 Cartridge Connector, SW1 SW_DIP_x04, SW2 SW_SPDT, U1 PRG ROM 512K, U2 CHR ROM 512K

Commit message: NROM x16: Refactor ROM bankswitching circuit
- Refactor routing
Parts:
- moved C3 1.95 mm to (63.5, 53.7), turned to 90 degrees
Connections:
- U2 pad 30: GND -> VCC
Routing:
- net /AUD_2A03: track 10.5 -> 0.00 mm
- net /CIRAM_~{CE}: track 10.5 -> 0.00 mm
- net /CPU_A8: track 30.8 -> 23.6 mm, vias 2 -> 1
- net /PPU_A12: track 52.8 -> 58.2 mm
- net /DIP_0: track 87.1 -> 92.2 mm
- net /PPU_A7: track 29.7 -> 25.4 mm, vias 3 -> 1
- net /PPU_D3: track 12.2 -> 16.3 mm
- net /DIP_1: track 89.7 -> 92.7 mm
- net GND: track 9.20 -> 6.51 mm, vias 45 -> 43
- net /PPU_A11: track 63.3 -> 60.8 mm
- net /PPU_A10: track 62.9 -> 60.9 mm
- net /CIRAM_A10: track 70.9 -> 69.0 mm
- net /PPU_~{RD}: track 56.3 -> 54.4 mm
- net /DIP_2: track 82.4 -> 84.1 mm
- net /CPU_A14: track 18.7 -> 17.4 mm, vias 1 -> 0
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